File: cad/rev3/delta-pico.kicad_pcb (KiCad board)
At the start: 2 copper layers, 77.7 x 159.8 mm, 73 parts, among them J1 Conn_01x02, J2 Conn_01x14, J3 Conn_01x04, J4 Conn_01x04, SW1 SW_SPDT, SW10 SW_Push, SW11 SW_Push, SW12 SW_Push, SW13 SW_Push, SW14 SW_Push, SW15 SW_Push, SW16 SW_Push, SW17 SW_Push, SW18 SW_Push, SW19 SW_Push, SW2 SW_Push, SW20 SW_Push, SW21 SW_Push, SW22 SW_Push, SW23 SW_Push, SW24 SW_Push, SW25 SW_Push, SW26 SW_Push, SW27 SW_Push, SW28 SW_Push, SW29 SW_Push, SW3 SW_Push, SW30 SW_Push, SW31 SW_Push, SW4 SW_Push, SW5 SW_Push, SW6 SW_Push, SW7 SW_Push, SW8 SW_Push, SW9 SW_Push, U1 PCF8574A, U2 PCF8574A, U3 Pico, U4 24LC16

Commit message: Update revision number silkscreen
Other:
- board text added: "Rev. 3"
- board text removed: "Rev. 2"
Changed lines of the file:
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@@
     (effects (font (size 2.3 2) (thickness 0.3)) (justify mirror))
   )
-  (gr_text "Rev. 2" (at 61.39 101.012) (layer "B.SilkS")
+  (gr_text "Rev. 3" (at 61.39 101.012) (layer "B.SilkS")
     (effects (font (size 1 1) (thickness 0.15)) (justify mirror))
   )

Commit message: Remove through-hole stuff from footprint, update board
Parts:
- U3: footprint MCU_RaspberryPi_and_Boards:RPi_Pico_SMD -> RPi_Pico:RPi_Pico_SMD_TH
Connections:
- J2 pad 10: Net-(J2-Pad10) -> unconnected-(J2-Pad10)
- J2 pad 11: Net-(J2-Pad11) -> unconnected-(J2-Pad11)
- J2 pad 12: Net-(J2-Pad12) -> unconnected-(J2-Pad12)
- J2 pad 13: Net-(J2-Pad13) -> unconnected-(J2-Pad13)
- J2 pad 14: Net-(J2-Pad14) -> unconnected-(J2-Pad14)
- SW1 pad 3: Net-(SW1-Pad3) -> unconnected-(SW1-Pad3)
- U1 pad 10: Net-(U1-Pad10) -> unconnected-(U1-Pad10)
- U1 pad 11: Net-(U1-Pad11) -> unconnected-(U1-Pad11)
- U1 pad 12: Net-(U1-Pad12) -> unconnected-(U1-Pad12)
- U1 pad 13: Net-(U1-Pad13) -> unconnected-(U1-Pad13)
- U2 pad 11: Net-(U2-Pad11) -> unconnected-(U2-Pad11)
- U2 pad 12: Net-(U2-Pad12) -> unconnected-(U2-Pad12)
- U2 pad 13: Net-(U2-Pad13) -> unconnected-(U2-Pad13)
- U3 pad 10: Net-(U3-Pad10) -> unconnected-(U3-Pad10)
- U3 pad 11: Net-(U3-Pad11) -> unconnected-(U3-Pad11)
- U3 pad 12: Net-(U3-Pad12) -> unconnected-(U3-Pad12)
- U3 pad 13: Net-(U3-Pad13) -> unconnected-(U3-Pad13)
- U3 pad 14: Net-(U3-Pad14) -> unconnected-(U3-Pad14)
- U3 pad 15: Net-(U3-Pad15) -> unconnected-(U3-Pad15)
- U3 pad 16: Net-(U3-Pad16) -> unconnected-(U3-Pad16)
- U3 pad 17: Net-(U3-Pad17) -> unconnected-(U3-Pad17)
- U3 pad 18: Net-(U3-Pad18) -> unconnected-(U3-Pad18)
- U3 pad 19: Net-(U3-Pad19) -> unconnected-(U3-Pad19)
- U3 pad 2: Net-(U3-Pad2) -> unconnected-(U3-Pad2)
- U3 pad 20: Net-(U3-Pad20) -> unconnected-(U3-Pad20)
- U3 pad 21: Net-(U3-Pad21) -> unconnected-(U3-Pad21)
- U3 pad 22: Net-(U3-Pad22) -> unconnected-(U3-Pad22)
- U3 pad 23: Net-(U3-Pad23) -> unconnected-(U3-Pad23)
- U3 pad 24: Net-(U3-Pad24) -> unconnected-(U3-Pad24)
- U3 pad 25: Net-(U3-Pad25) -> unconnected-(U3-Pad25)
- U3 pad 28: Net-(U3-Pad28) -> unconnected-(U3-Pad28)
- U3 pad 29: Net-(U3-Pad29) -> unconnected-(U3-Pad29)
- U3 pad 30: Net-(U3-Pad30) -> unconnected-(U3-Pad30)
- U3 pad 31: Net-(U3-Pad31) -> unconnected-(U3-Pad31)
- U3 pad 32: Net-(U3-Pad32) -> unconnected-(U3-Pad32)
- U3 pad 33: Net-(U3-Pad33) -> unconnected-(U3-Pad33)
- U3 pad 35: Net-(U3-Pad35) -> unconnected-(U3-Pad35)
- U3 pad 37: Net-(U3-Pad37) -> unconnected-(U3-Pad37)
- U3 pad 38: Net-(U3-Pad38) -> unconnected-(U3-Pad38)
- U3 pad 40: Net-(U3-Pad40) -> unconnected-(U3-Pad40)
- U3 pad 41: Net-(U3-Pad41) -> unconnected-(U3-Pad41)
- U3 pad 42: Net-(U3-Pad42) -> unconnected-(U3-Pad42)
- U3 pad 43: Net-(U3-Pad43) -> unconnected-(U3-Pad43)
- U3 pad 8: Net-(U3-Pad8) -> unconnected-(U3-Pad8)

Commit message: Fix a lot of DRC errors
Routing:
- net SD_CS: track 19.7 -> 17.1 mm
- net ROW0: track 90.9 -> 89.1 mm
- net GND: track 246.8 -> 246.2 mm
Changed lines of the file:
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@@
   (gr_line (start 111.2 33.05) (end 111.2 182.25) (layer "Edge.Cuts") (width 0.05))
   (gr_arc (start 105.896228 27.746228) (mid 109.646561 29.299667) (end 111.2 33.05) (layer "Edge.Cuts") (width 0.05))
-  (gr_arc (start 111.203772 182.25) (mid 109.650333 186.000333) (end 105.9 187.553772) (layer "Edge.Cuts") (width 0.05))
+  (gr_arc (start 111.2 182.25) (mid 109.648998 186.000102) (end 105.9 187.553772) (layer "Edge.Cuts") (width 0.05))
   (gr_line (start 38.8 27.746228) (end 105.896228 27.746228) (layer "Edge.Cuts") (width 0.05))
   (gr_line (start 38.803772 187.553772) (end 105.9 187.55) (layer "Edge.Cuts") (width 0.05))
@@
   (segment (start 88.826 138.822) (end 90.35 140.346) (width 0.25) (layer "B.Cu") (net 2))
   (segment (start 86.28399 127.38999) (end 82.095 123.201) (width 0.25) (layer "B.Cu") (net 2))
-  (segment (start 104.828 140.346) (end 106.606 140.346) (width 0.25) (layer "B.Cu") (net 2))
   (segment (start 76.126 140.346) (end 79.428 140.346) (width 0.25) (layer "B.Cu") (net 2))
   (segment (start 93.906 131.202) (end 90.09399 127.38999) (width 0.25) (layer "B.Cu") (net 2))
@@
   (segment (start 87.175 119.44) (end 87.175 118.415) (width 0.25) (layer "B.Cu") (net 37))
   (segment (start 55.499 41.783) (end 63.5 33.782) (width 0.25) (layer "B.Cu") (net 37))
-  (segment (start 99.7966 34.6964) (end 99.2251 34.6964) (width 0.25) (layer "B.Cu") (net 37))
   (segment (start 63.33 119.44) (end 62.49 119.44) (width 0.25) (layer "B.Cu") (net 37))
   (segment (start 52.959 49.719) (end 52.959 44.769) (width 0.25) (layer "B.Cu") (net 37))
@@
   (segment (start 75.92 106.73) (end 89.75 92.9) (width 0.25) (layer "B.Cu") (net 44))
   (segment (start 104.8639 29.6164) (end 99.7966 29.6164) (width 0.25) (layer "B.Cu") (net 44))
+  (segment (start 79.3736 39.7764) (end 82.0166 39.7764) (width 0.25) (layer "F.Cu") (net 45))
   (segment (start 62.9 128.2) (end 60.4 125.7) (width 0.25) (layer "F.Cu") (net 45))
   (segment (start 77.315 117.2) (end 76.33 117.2) (width 0.25) (layer "F.Cu") (net 45))
@@
   (segment (start 79.555 119.44) (end 77.315 117.2) (width 0.25) (layer "F.Cu") (net 45))
   (segment (start 76.33 117.2) (end 73.38 114.25) (width 0.25) (layer "F.Cu") (net 45))
-  (segment (start 79.3736 39.7764) (end 82.0166 39.7764) (width 0.25) (layer "F.Cu") (net 45))
   (segment (start 55.6 86.81) (end 36.7284 67.9384) (width 0.25) (layer "F.Cu") (net 45))
   (segment (start 78.412 128.613) (end 78.285 128.74) (width 0.25) (layer "F.Cu") (net 45))
-  (via (at 82.0166 39.7764) (size 0.8) (drill 0.4) (layers "F.Cu" "B.Cu") (net 45))
   (via (at 79.555 119.44) (size 0.8) (drill 0.4) (layers "F.Cu" "B.Cu") (net 45))
   (via (at 51.816 47.498) (size 0.8) (drill 0.4) (layers "F.Cu" "B.Cu") (net 45))
+  (via (at 82.0166 39.7764) (size 0.8) (drill 0.4) (layers "F.Cu" "B.Cu") (net 45))
   (via (at 78.285 128.74) (size 0.8) (drill 0.4) (layers "F.Cu" "B.Cu") (net 45))
   (via (at 60.3 125.7) (size 0.8) (drill 0.4) (layers "F.Cu" "B.Cu") (net 45))
@@
   (segment (start 51.689 49.719) (end 51.689 47.625) (width 0.25) (layer "B.Cu") (net 45))
   (segment (start 43.75 57.658) (end 40.64 57.658) (width 0.25) (layer "B.Cu") (net 45))
-  (segment (start 81.8642 39.624) (end 82.0166 39.7764) (width 0.25) (layer "B.Cu") (net 45))
   (segment (start 64.569 128.74) (end 64.569 129.765) (width 0.25) (layer "B.Cu") (net 45))
   (segment (start 64.569 128.74) (end 63.44 128.74) (width 0.25) (layer "B.Cu") (net 45))
@@
   (segment (start 50.24 32.26) (end 81.913 32.26) (width 0.25) (layer "B.Cu") (net 52))
   (segment (start 38.6 43.9) (end 50.24 32.26) (width 0.25) (layer "B.Cu") (net 52))
-  (segment (start 46.99 160.66) (end 46.92 160.73) (width 0.25) (layer "F.Cu") (net 53))
-  (segment (start 46.89 169.43) (end 46.86 169.46) (width 0.25) (layer "F.Cu") (net 53))
-  (segment (start 46.83 178.21) (end 46.81 178.23) (width 0.25) (layer "F.Cu") (net 53))
   (segment (start 46.86 169.46) (end 46.86 160.79) (width 0.25) (layer "F.Cu") (net 53))
   (segment (start 46.92 160.73) (end 46.92 152) (width 0.25) (layer "F.Cu") (net 53))
   (segment (start 47.02 151.9) (end 46.120001 151.000001) (width 0.25) (layer "F.Cu") (net 53))
   (segment (start 44.122 133.946) (end 50.572 133.946) (width 0.25) (layer "F.Cu") (net 53))
-  (segment (start 46.92 152) (end 47.02 151.9) (width 0.25) (layer "F.Cu") (net 53))
   (segment (start 46.86 160.79) (end 46.92 160.73) (width 0.25) (layer "F.Cu") (net 53))
-  (segment (start 46.81 169.51) (end 46.86 169.46) (width 0.25) (layer "F.Cu") (net 53))
   (segment (start 50.572 133.946) (end 54.332 130.186) (width 0.25) (layer "F.Cu") (net 53))
-  (segment (start 47.04 151.88) (end 47.02 151.9) (width 0.25) (layer "F.Cu") (net 53))
   (segment (start 46.120001 135.944001) (end 44.122 133.946) (width 0.25) (layer "F.Cu") (net 53))
   (segment (start 46.120001 151.000001) (end 46.120001 135.944001) (width 0.25) (layer "F.Cu") (net 53))
@@
   (segment (start 61.38 151.92) (end 54.332 144.872) (width 0.25) (layer "F.Cu") (net 54))
   (segment (start 61.27 169.47) (end 61.26 169.48) (width 0.25) (layer "F.Cu") (net 54))
-  (segment (start 61.29 160.74) (end 61.27 160.72) (width 0.25) (layer "F.Cu") (net 54))
   (segment (start 54.332 137.706) (end 58.092 133.946) (width 0.25) (layer "F.Cu") (net 54))
-  (segment (start 61.35 160.64) (end 61.27 160.72) (width 0.25) (layer "F.Cu") (net 54))
   (segment (start 61.38 160.61) (end 61.27 160.72) (width 0.25) (layer "F.Cu") (net 54))
   (segment (start 54.332 143.902) (end 54.332 137.706) (width 0.25) (layer "F.Cu") (net 54))
@@
   (segment (start 58.092 131.423768) (end 69.649 119.866768) (width 0.25) (layer "B.Cu") (net 54))
   (segment (start 69.649 119.866768) (end 69.649 119.44) (width 0.25) (layer "B.Cu") (net 54))
-  (segment (start 75.71 169.45) (end 75.74 169.48) (width 0.25) (layer "F.Cu") (net 55))
   (segment (start 75.85 151.88) (end 75.8 151.93) (width 0.25) (layer "F.Cu") (net 55))
   (segment (start 75.85 134.38) (end 75.85 143.16) (width 0.25) (layer "F.Cu") (net 55))
-  (segment (start 75.69 169.53) (end 75.74 169.48) (width 0.25) (layer "F.Cu") (net 55))
   (segment (start 75.85 143.16) (end 75.85 151.88) (width 0.25) (layer "F.Cu") (net 55))
   (segment (start 75.85 134.38) (end 72.7 134.38) (width 0.25) (layer "F.Cu") (net 55))
   (segment (start 70.919 132.599) (end 70.919 119.44) (width 0.25) (layer "F.Cu") (net 55))
-  (segment (start 75.71 178.23) (end 75.69 178.25) (width 0.25) (layer "F.Cu") (net 55))
   (segment (start 75.74 169.48) (end 75.74 160.72) (width 0.25) (layer "F.Cu") (net 55))
   (segment (start 75.74 160.72) (end 75.74 151.99) (width 0.25) (layer "F.Cu") (net 55))
   (segment (start 75.74 151.99) (end 75.8 151.93) (width 0.25) (layer "F.Cu") (net 55))
-  (segment (start 75.77 160.69) (end 75.74 160.72) (width 0.25) (layer "F.Cu") (net 55))
   (segment (start 72.7 134.38) (end 70.919 132.599) (width 0.25) (layer "F.Cu") (net 55))
   (segment (start 75.69 178.25) (end 75.69 169.53) (width 0.25) (layer "F.Cu") (net 55))
@@
   (segment (start 90.28 134.49) (end 87.5 131.71) (width 0.25) (layer "F.Cu") (net 56))
   (segment (start 90.28 134.49) (end 90.28 143.26) (width 0.25) (layer "F.Cu") (net 56))
-  (segment (start 90.11 169.59) (end 90.12 169.58) (width 0.25) (layer "F.Cu") (net 56))
   (segment (start 90.12 178.3) (end 90.08 178.34) (width 0.25) (layer "F.Cu") (net 56))
   (segment (start 72.189 129.043) (end 72.189 119.44) (width 0.25) (layer "F.Cu") (net 56))
-  (segment (start 90.1 169.56) (end 90.12 169.58) (width 0.25) (layer "F.Cu") (net 56))
-  (segment (start 90.13 169.57) (end 90.12 169.58) (width 0.25) (layer "F.Cu") (net 56))
   (segment (start 90.26 160.68) (end 90.13 160.81) (width 0.25) (layer "F.Cu") (net 56))
   (segment (start 90.28 143.26) (end 90.28 152.03) (width 0.25) (layer "F.Cu") (net 56))
   (via (at 72.189 119.44) (size 0.8) (drill 0.4) (layers "F.Cu" "B.Cu") (net 56))
   (segment (start 104.74 134.49) (end 100.944 130.694) (width 0.25) (layer "F.Cu") (net 57))
-  (segment (start 104.63 152.13) (end 104.71 152.05) (width 0.25) (layer "F.Cu") (net 57))
   (segment (start 100.944 130.694) (end 75.413 130.694) (width 0.25) (layer "F.Cu") (net 57))
   (segment (start 104.6 169.57) (end 104.6 160.82) (width 0.25) (layer "F.Cu") (net 57))
@@
   (segment (start 104.54 178.36) (end 104.54 169.63) (width 0.25) (layer "F.Cu") (net 57))
   (segment (start 75.413 130.694) (end 73.459 128.74) (width 0.25) (layer "F.Cu") (net 57))
-  (segment (start 104.74 152.02) (end 104.71 152.05) (width 0.25) (layer "F.Cu") (net 57))
   (segment (start 104.71 152.05) (end 104.71 143.28) (width 0.25) (layer "F.Cu") (net 57))
   (segment (start 104.74 143.25) (end 104.74 134.49) (width 0.25) (layer "F.Cu") (net 57))
   (segment (start 104.54 169.63) (end 104.6 169.57) (width 0.25) (layer "F.Cu") (net 57))
-  (segment (start 104.68 160.74) (end 104.63 160.79) (width 0.25) (layer "F.Cu") (net 57))
-  (segment (start 104.57 178.33) (end 104.54 178.36) (width 0.25) (layer "F.Cu") (net 57))
-  (segment (start 104.6 160.82) (end 104.63 160.79) (width 0.25) (layer "F.Cu") (net 57))
   (segment (start 104.63 160.79) (end 104.63 152.13) (width 0.25) (layer "F.Cu") (net 57))
   (via (at 73.459 128.74) (size 0.8) (drill 0.4) (layers "F.Cu" "B.Cu") (net 57))
@@
   (segment (start 82.0166 44.8564) (end 76.6664 44.8564) (width 0.25) (layer "B.Cu") (net 67))
   (segment (start 76.6664 44.8564) (end 68.35 36.54) (width 0.25) (layer "B.Cu") (net 67))
-  (segment (start 82.0166 44.8564) (end 79.4434 44.8564) (width 0.25) (layer "B.Cu") (net 67))
   (zone (net 0) (net_name "") (layer "B.Cu") (hatch edge 0.508)
     (connect_pads (clearance 0))
